Commit message: calibration on exp data

File: scripts/models/robots/tiago_description/robots/tiago_no_hand_mod.urdf (robot description, URDF)
Before this commit: robot tiago, 39 links, 38 joints
Links:
- removed link ee_marker
- added link ee_marker_link, mass 0.0
Joints:
- joint ee_marker_joint: child ee_marker -> ee_marker_link; type revolute -> fixed
