Commit message: correct urdf full talos

File: scripts/models/others/robots/talos_data/robots/talos_full_v2.urdf (robot description, URDF)
Before this commit: robot talos, 60 links, 59 joints
Links:
- link arm_left_1_link: geometry collision mesh filename=package://talos_description/meshes/arm/arm_1_collision.STL scale=1 1 1; visual mesh filename=package://talos_description/meshes/arm/arm_1.STL scale=1 1 1
- link arm_left_2_link: geometry collision mesh filename=package://talos_description/meshes/arm/arm_2_collision.STL scale=1 1 1; visual mesh filename=package://talos_description/meshes/arm/arm_2.STL scale=1 1 1
- link arm_left_3_link: geometry collision mesh filename=package://talos_description/meshes/arm/arm_3_collision.STL scale=1 1 1; visual mesh filename=package://talos_description/meshes/arm/arm_3.STL scale=1 1 1
- link arm_left_4_link: geometry collision mesh filename=package://talos_description/meshes/arm/arm_4_collision.STL scale=1 1 1; visual mesh filename=package://talos_description/meshes/arm/arm_4.STL scale=1 1 1
- link arm_left_5_link: geometry collision mesh filename=package://talos_description/meshes/arm/arm_5_collision.STL scale=1 1 1; visual mesh filename=package://talos_description/meshes/arm/arm_5.STL scale=1 1 1
- link arm_left_6_link: geometry collision mesh filename=package://talos_description/meshes/arm/arm_6_collision.STL scale=1 1 1; visual mesh filename=package://talos_description/meshes/arm/arm_6.STL scale=1 1 1
- link arm_left_7_link: geometry collision mesh filename=package://talos_description/meshes/arm/arm_7_collision.STL scale=1 1 1; visual mesh filename=package://talos_description/meshes/arm/arm_7.STL scale=1 1 1
- link arm_right_1_link: geometry collision mesh filename=package://talos_description/meshes/arm/arm_1_collision.STL scale=1 -1 1; visual mesh filename=package://talos_description/meshes/arm/arm_1.STL scale=1 -1 1
- link arm_right_2_link: geometry collision mesh filename=package://talos_description/meshes/arm/arm_2_collision.STL scale=1 -1 1; visual mesh filename=package://talos_description/meshes/arm/arm_2.STL scale=1 -1 1
- link arm_right_3_link: geometry collision mesh filename=package://talos_description/meshes/arm/arm_3_collision.STL scale=1 -1 1; visual mesh filename=package://talos_description/meshes/arm/arm_3.STL scale=1 -1 1
- link arm_right_4_link: geometry collision mesh filename=package://talos_description/meshes/arm/arm_4_collision.STL scale=1 -1 1; visual mesh filename=package://talos_description/meshes/arm/arm_4.STL scale=1 -1 1
- link arm_right_5_link: geometry collision mesh filename=package://talos_description/meshes/arm/arm_5_collision.STL scale=1 -1 1; visual mesh filename=package://talos_description/meshes/arm/arm_5.STL scale=1 -1 1
- link arm_right_6_link: geometry collision mesh filename=package://talos_description/meshes/arm/arm_6_collision.STL scale=1 -1 1; visual mesh filename=package://talos_description/meshes/arm/arm_6.STL scale=1 -1 1
- link arm_right_7_link: geometry collision mesh filename=package://talos_description/meshes/arm/arm_7_collision.STL scale=1 -1 1; visual mesh filename=package://talos_description/meshes/arm/arm_7.STL scale=1 -1 1
- link base_link: geometry collision mesh filename=package://talos_description/meshes/torso/base_link_collisio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 scale=1 1 1; visual mesh filename=package://talos_description/meshes/torso/base_link.STL scale=1 1 1
- link gripper_left_base_link: mass 0.61585 -> 0.637534; geometry collision mesh filename=package://talos_description/meshes/gripper/base_link_collis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 scale=1 1 1; visual mesh filename=package://talos_description/meshes/gripper/base_link.STL scale=1 1 1
- link gripper_left_fingertip_1_link: mass 0.02630 -> 0.026301; geometry collision mesh filename=package://talos_description/meshes/gripper/fingertip_collis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 scale=1 1 1; visual mesh filename=package://talos_description/meshes/gripper/fingertip.STL scale=1 1 1
- link gripper_left_fingertip_2_link: mass 0.02630 -> 0.026301; geometry collision mesh filename=package://talos_description/meshes/gripper/fingertip_collis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 scale=1 1 1; visual mesh filename=package://talos_description/meshes/gripper/fingertip.STL scale=1 1 1
- link gripper_left_fingertip_3_link: mass 0.02630 -> 0.026301; geometry collision mesh filename=package://talos_description/meshes/gripper/fingertip_collis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 scale=1 1 1; visual mesh filename=package://talos_description/meshes/gripper/fingertip.STL scale=1 1 1
- link gripper_left_inner_double_link: mass 0.11922 -> 0.087986; geometry collision mesh filename=package://talos_description/meshes/gripper/inner_double_col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 scale=1 1 1; visual mesh filename=package://talos_description/meshes/gripper/inner_double.STL scale=1 1 1
- link gripper_left_inner_single_link: mass 0.05356 -> 0.047177; geometry collision mesh filename=package://talos_description/meshes/gripper/inner_single_col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 scale=1 1 1; visual mesh filename=package://talos_description/meshes/gripper/inner_single.STL scale=1 1 1
- link gripper_left_motor_double_link: mass 0.16889 -> 0.134356; geometry collision mesh filename=package://talos_description/meshes/gripper/gripper_motor_do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 scale=1 1 1; visual mesh filename=package://talos_description/meshes/gripper/gripper_motor_do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 scale=1 1 1
- link gripper_left_motor_single_link: mass 0.14765 -> 0.107923; geometry collision mesh filename=package://talos_description/meshes/gripper/gripper_motor_si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 scale=1 1 1; visual mesh filename=package://talos_description/meshes/gripper/gripper_motor_si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 scale=1 1 1
- link gripper_right_base_link: mass 0.61585 -> 0.637534; geometry collision mesh filename=package://talos_description/meshes/gripper/base_link_collis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 scale=1 1 1; visual mesh filename=package://talos_description/meshes/gripper/base_link.STL scale=1 1 1
- link gripper_right_fingertip_1_link: mass 0.02630 -> 0.026301; geometry collision mesh filename=package://talos_description/meshes/gripper/fingertip_collis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 scale=1 1 1; visual mesh filename=package://talos_description/meshes/gripper/fingertip.STL scale=1 1 1
- link gripper_right_fingertip_2_link: mass 0.02630 -> 0.026301; geometry collision mesh filename=package://talos_description/meshes/gripper/fingertip_collis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 scale=1 1 1; visual mesh filename=package://talos_description/meshes/gripper/fingertip.STL scale=1 1 1
- link gripper_right_fingertip_3_link: mass 0.02630 -> 0.026301; geometry collision mesh filename=package://talos_description/meshes/gripper/fingertip_collis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 scale=1 1 1; visual mesh filename=package://talos_description/meshes/gripper/fingertip.STL scale=1 1 1
- link gripper_right_inner_double_link: mass 0.11922 -> 0.087986; geometry collision mesh filename=package://talos_description/meshes/gripper/inner_double_col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 scale=1 1 1; visual mesh filename=package://talos_description/meshes/gripper/inner_double.STL scale=1 1 1
- link gripper_right_inner_single_link: mass 0.05356 -> 0.047177; geometry collision mesh filename=package://talos_description/meshes/gripper/inner_single_col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 scale=1 1 1; visual mesh filename=package://talos_description/meshes/gripper/inner_single.STL scale=1 1 1
- link gripper_right_motor_double_link: mass 0.16889 -> 0.134356; geometry collision mesh filename=package://talos_description/meshes/gripper/gripper_motor_do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 scale=1 1 1; visual mesh filename=package://talos_description/meshes/gripper/gripper_motor_do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 scale=1 1 1
- link gripper_right_motor_single_link: mass 0.14765 -> 0.107923; geometry collision mesh filename=package://talos_description/meshes/gripper/gripper_motor_si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 scale=1 1 1; visual mesh filename=package://talos_description/meshes/gripper/gripper_motor_si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 scale=1 1 1
- link head_1_link: mass 0.65988 -> 0.73746; geometry collision mesh filename=package://talos_description/meshes/head/head_1_collision.stl scale=1 1 1; visual mesh filename=package://talos_description/meshes/head/head_1.stl scale=1 1 1
- link head_2_link: mass 1.40353 -> 1.443954; geometry collision mesh filename=package://talos_description/meshes/head/head_2_collision.stl scale=1 1 1; visual mesh filename=package://talos_description/meshes/head/head_2.stl scale=1 1 1
- link leg_left_1_link: mass 1.88569 -> 1.845591; geometry collision mesh filename=package://talos_description/meshes/v2/hip_z_collision.stl scale=1 1 1; visual mesh filename=package://talos_description/meshes/v2/hip_z_lo_res.stl scale=1 1 1
- link leg_left_2_link: mass 2.37607 -> 1.490952; geometry collision mesh filename=package://talos_description/meshes/v2/hip_x_collision.stl scale=1 1 1; visual mesh filename=package://talos_description/meshes/v2/hip_x_lo_res.stl scale=1 1 1
- link leg_left_3_link: mass 6.82734 -> 6.239871; geometry collision mesh filename=package://talos_description/meshes/v2/hip_y_collision.stl scale=1 1 1; visual mesh filename=package://talos_description/meshes/v2/hip_y_lo_res.stl scale=1 1 1
- link leg_left_4_link: mass 3.63668 -> 3.759951; geometry collision mesh filename=package://talos_description/meshes/v2/knee_collision.stl scale=1 1 1; visual mesh filename=package://talos_description/meshes/v2/knee_lo_res.stl scale=1 1 1
- link leg_left_5_link: mass 1.24433 -> 1.29096; geometry collision mesh filename=package://talos_description/meshes/v2/ankle_Y_collision.stl scale=1 1 1; visual mesh filename=package://talos_description/meshes/v2/ankle_Y_lo_res.stl scale=1 1 1
- link leg_left_6_link: mass 1.59457 -> 1.597773; geometry collision mesh filename=package://talos_description/meshes/v2/ankle_X_collision.stl scale=1.15 1.05 1; visual mesh filename=package://talos_description/meshes/v2/ankle_X_lo_res.stl scale=1 1 1
- link leg_right_1_link: mass 1.88569 -> 1.845591; geometry collision mesh filename=package://talos_description/meshes/v2/hip_z_collision.stl scale=1 -1 1; visual mesh filename=package://talos_description/meshes/v2/hip_z_lo_res.stl scale=1 -1 1
- link leg_right_2_link: mass 2.37607 -> 1.490952; geometry collision mesh filename=package://talos_description/meshes/v2/hip_x_collision.stl scale=1 -1 1; visual mesh filename=package://talos_description/meshes/v2/hip_x_lo_res.stl scale=1 -1 1
- link leg_right_3_link: mass 6.82734 -> 6.239871; geometry collision mesh filename=package://talos_description/meshes/v2/hip_y_collision.stl scale=1 -1 1; visual mesh filename=package://talos_description/meshes/v2/hip_y_lo_res.stl scale=1 -1 1
- link leg_right_4_link: mass 3.63668 -> 3.759951; geometry collision mesh filename=package://talos_description/meshes/v2/knee_collision.stl scale=1 -1 1; visual mesh filename=package://talos_description/meshes/v2/knee_lo_res.stl scale=1 -1 1
- link leg_right_5_link: mass 1.24433 -> 1.29096; geometry collision mesh filename=package://talos_description/meshes/v2/ankle_Y_collision.stl scale=1 -1 1; visual mesh filename=package://talos_description/meshes/v2/ankle_Y_lo_res.stl scale=1 -1 1
- link leg_right_6_link: mass 1.59457 -> 1.597773; geometry collision mesh filename=package://talos_description/meshes/v2/ankle_X_collision.stl scale=1.15 -1.05 1; visual mesh filename=package://talos_description/meshes/v2/ankle_X_lo_res.stl scale=1 -1 1
- link rgbd_link: geometry collision box size=0.04 0.185 0.03; visual mesh filename=package://talos_description/meshes/sensors/orbbec/orbbec.STL
- link torso_1_link: geometry collision mesh filename=package://talos_description/meshes/torso/torso_1.STL scale=1 1 1; visual mesh filename=package://talos_description/meshes/torso/torso_1.STL scale=1 1 1
- link torso_2_link: mass 17.55011 -> 16.97403; geometry collision mesh filename=package://talos_description/meshes/torso/torso_2_collision.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 scale=1 1 1; visual mesh filename=package://talos_description/meshes/torso/torso_2.STL scale=1 1 1
- link wrist_left_ft_link: mass 0.1 -> 0.095
- link wrist_left_ft_tool_link: mass 0.1 -> 0.001
- link wrist_right_ft_link: mass 0.1 -> 0.095
- link wrist_right_ft_tool_link: mass 0.1 -> 0.001
Joints:
- joint gripper_left_joint: limit lower=-1.0471975512 upper=0.0 effort=1.0 velocity=1.0 -> lower=-0.959931088597 upper=0.0 effort=1.0 velocity=1.0
- joint gripper_right_joint: limit lower=-1.0471975512 upper=0.0 effort=1.0 velocity=1.0 -> lower=-0.959931088597 upper=0.0 effort=1.0 velocity=1.0
- joint head_1_joint: limit lower=-0.261799387799 upper=0.785398163397 effort=8.0 velocity=1.0 -> lower=-0.209439510239 upper=0.785398163397 effort=8.0 velocity=3.0; origin xyz=0.00000 0.00000 0.31600 rpy=0.0 0.0 0.0 -> xyz=0.02000 0.00000 0.32100 rpy=0.0 0.0 0.0
- joint head_2_joint: limit lower=-1.308996939 upper=1.308996939 effort=4.0 velocity=1.0 -> lower=-1.308996939 upper=1.308996939 effort=4.0 velocity=3.0
- joint imu_joint: origin xyz=0.04925 0 0.078 rpy=3.14159265359 0 1.57079632679 -> xyz=0.04925 0.0 0.078 rpy=3.14159265359 0.0 1.57079632679
- joint leg_left_4_joint: limit lower=0 upper=2.618 effort=300 velocity=7 -> lower=0 upper=2.618 effort=400 velocity=7
- joint leg_left_5_joint: limit lower=-1.309 upper=0.768 effort=160 velocity=5.8 -> lower=-1.27 upper=0.68 effort=160 velocity=5.8
- joint leg_right_4_joint: limit lower=0 upper=2.618 effort=300 velocity=7 -> lower=0 upper=2.618 effort=400 velocity=7
- joint leg_right_5_joint: limit lower=-1.309 upper=0.768 effort=160 velocity=5.8 -> lower=-1.27 upper=0.68 effort=160 velocity=5.8
- joint rgbd_joint: origin xyz=0.066 0.0 0.1982 rpy=0 0 0 -> xyz=0.066 0.0 0.1982 rpy=0.0 0.0 0.0
