Commit message: re-correct urdf talos_reduced

File: scripts/models/others/robots/talos_data/robots/talos_reduced.urdf (robot description, URDF)
Before this commit: robot talos, 60 links, 59 joints
Links:
- link torso_2_link: mass 17.55011 -> 16.97403
Joints:
- joint imu_joint: origin xyz=0.04925 0 0.078 rpy=3.14159265359 0 1.57079632679 -> xyz=0.04925 0.0 0.078 rpy=3.14159265359 0.0 1.57079632679
